File: Hardware/LSM9DS1/LSM9DS1.brd (EAGLE design)
At the start: 20.3 x 13 mm, 11 parts, among them U1 LSM9DS1

Commit message: Rev 3 IMU Board
Here it is, in all its glory.
Parts:
- added D1: BLUE, SparkFun-LED:LED-0603
- added R2: (no value), SparkFun-Passives:0603-RES
- moved C4 0.08 mm to (16.5, 8.33)
- moved C5 0.08 mm to (14.4, 8.33)
- renumbered JP3 to JP1
Connections:
- net CSCLK: now also JP1.2; no longer JP1.7
- net CS_A/G: now also D1.C
- net CS_M: now also R2.2
- net D: now also JP1.6; no longer JP1.3
- net GND: now also JP1.7, JP1.8; no longer JP1.1, JP1.2
- net SCL: now also JP1.3; no longer JP1.6
- net SDA: now also JP1.4; no longer JP1.5
- net SDO_A/G: now also JP1.5; no longer JP1.4
- net VDD: now also D1.A, JP1.1, R2.1; no longer JP1.8
Routing:
- net CSCLK: track 17.5 -> 9.62 mm
- net CS_A/G: track 14.7 -> 22.0 mm, vias 3 -> 5
- net SCL: track 18.7 -> 14.0 mm
- net D: track 5.25 -> 8.61 mm
- net CS_M: track 8.73 -> 11.0 mm, vias 0 -> 1
- net GND: track 7.64 -> 5.64 mm
- net VDD: track 33.3 -> 31.4 mm
- net SDA: track 15.1 -> 13.4 mm
- net N$2: track 2.47 -> 3.26 mm
- net SDO_A/G: track 13.7 -> 12.9 mm
