File: Hardware/LSM9DS1/LSM9DS1.sch (EAGLE design)
At the start: 11 parts, among them U1 LSM9DS1

Commit message: Rev 3 IMU Board
Here it is, in all its glory.
Parts:
- removed JP3: (no value), SparkFun-Connectors:M08BM08B-SRSS-TB
- added D1: BLUE, SparkFun-LED:LED-BLUE0603
- added JP1: (no value), SparkFun-Connectors:M08BM08B-SRSS-TB
- added R2: (no value), SparkFun-Passives:RESISTOR0603-RES
Connections:
- net CSCLK: now also JP1.2; no longer JP3.7
- net CS_A/G: now also D1.C
- net CS_M: now also R2.2
- net D: now also JP1.6; no longer JP3.3
- net GND: now also JP1.7, JP1.8; no longer JP3.1, JP3.2
- net SCL: now also JP1.3; no longer JP3.6
- net SDA: now also JP1.4; no longer JP3.5
- net SDO_A/G: now also JP1.5; no longer JP3.4
- net VDD: now also D1.A, JP1.1, R2.1; no longer JP3.8
Changed lines of the file:
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@@
 <?xml version="1.0" encoding="utf-8"?>
 <!DOCTYPE eagle SYSTEM "eagle.dtd">
-<eagle version="7.2.0">
+<eagle version="7.4.0">
 <drawing>
 <settings>
@@
 <part name="R1" library="SparkFun-Passives" deviceset="RESISTOR" device="0603-RES"/>
 <part name="JP2" library="SparkFun-Connectors" deviceset="M08" device="BM08B-SRSS-TB"/>
-<part name="JP3" library="SparkFun-Connectors" deviceset="M08" device="BM08B-SRSS-TB"/>
 <part name="JP4" library="SparkFun-Connectors" deviceset="M08" device="BM08B-SRSS-TB"/>
 <part name="SUPPLY4" library="SparkFun-Aesthetics" deviceset="VDD" device=""/>
 <part name="GND3" library="SparkFun-Aesthetics" deviceset="GND" device=""/>
+<part name="JP1" library="SparkFun-Connectors" deviceset="M08" device="BM08B-SRSS-TB"/>
+<part name="D1" library="SparkFun-LED" deviceset="LED-BLUE" device="0603" value="BLUE"/>
+<part name="R2" library="SparkFun-Passives" deviceset="RESISTOR" device="0603-RES"/>
+<part name="SUPPLY1" library="SparkFun-Aesthetics" deviceset="VDD" device=""/>
 </parts>
 <sheets>
@@
 <instance part="R1" gate="G$1" x="96.52" y="106.68" rot="R180"/>
 <instance part="JP2" gate="G$1" x="144.78" y="81.28"/>
-<instance part="JP3" gate="G$1" x="170.18" y="81.28" rot="MR0"/>
 <instance part="JP4" gate="G$1" x="149.86" y="40.64" rot="R180"/>
 <instance part="SUPPLY4" gate="VDD" x="157.48" y="93.98"/>
 <instance part="GND3" gate="1" x="157.48" y="68.58"/>
+<instance part="JP1" gate="G$1" x="170.18" y="83.82" rot="R180"/>
+<instance part="D1" gate="G$1" x="104.14" y="99.06"/>
+<instance part="R2" gate="G$1" x="93.98" y="71.12" rot="R270"/>
+<instance part="SUPPLY1" gate="VDD" x="93.98" y="78.74"/>
 </instances>
 <busses>
@@
 <wire x1="104.14" y1="106.68" x2="104.14" y2="114.3" width="0.1524" layer="91"/>
 <junction x="104.14" y="106.68"/>
+<pinref part="D1" gate="G$1" pin="A"/>
+<junction x="104.14" y="101.6"/>
 </segment>
 <segment>
 <pinref part="JP2" gate="G$1" pin="8"/>
-<pinref part="JP3" gate="G$1" pin="8"/>
 <wire x1="149.86" y1="91.44" x2="157.48" y2="91.44" width="0.1524" layer="91"/>
 <wire x1="157.48" y1="91.44" x2="165.1" y2="91.44" width="0.1524" layer="91"/>
@@
 <pinref part="SUPPLY4" gate="VDD" pin="VDD"/>
 <junction x="157.48" y="91.44"/>
+<pinref part="JP1" gate="G$1" pin="1"/>
+</segment>
+<segment>
+<pinref part="R2" gate="G$1" pin="1"/>
+<pinref part="SUPPLY1" gate="VDD" pin="VDD"/>
+<wire x1="93.98" y1="76.2" x2="93.98" y2="78.74" width="0.1524" layer="91"/>
 </segment>
 </net>
@@
 </segment>
 <segment>
-<pinref part="JP3" gate="G$1" pin="1"/>
 <pinref part="JP2" gate="G$1" pin="1"/>
 <wire x1="165.1" y1="73.66" x2="157.48" y2="73.66" width="0.1524" layer="91"/>
@@
 <wire x1="157.48" y1="73.66" x2="157.48" y2="71.12" width="0.1524" layer="91"/>
 <pinref part="GND3" gate="1" pin="GND"/>
-<pinref part="JP3" gate="G$1" pin="2"/>
 <pinref part="JP2" gate="G$1" pin="2"/>
 <wire x1="165.1" y1="76.2" x2="157.48" y2="76.2" width="0.1524" layer="91"/>
@@
 <junction x="157.48" y="76.2"/>
 <junction x="157.48" y="73.66"/>
+<pinref part="JP1" gate="G$1" pin="7"/>
+<pinref part="JP1" gate="G$1" pin="8"/>
 </segment>
 </net>
@@
 <segment>
 <pinref part="JP2" gate="G$1" pin="6"/>
-<pinref part="JP3" gate="G$1" pin="6"/>
 <wire x1="149.86" y1="86.36" x2="165.1" y2="86.36" width="0.1524" layer="91"/>
 <label x="152.4" y="86.36" size="1.778" layer="95"/>
+<pinref part="JP1" gate="G$1" pin="3"/>
 </segment>
 </net>
@@
 <segment>
 <pinref part="JP2" gate="G$1" pin="5"/>
-<pinref part="JP3" gate="G$1" pin="5"/>
 <wire x1="149.86" y1="83.82" x2="165.1" y2="83.82" width="0.1524" layer="91"/>
+<pinref part="JP1" gate="G$1" pin="4"/>
 </segment>
 </net>
@@
 <segment>
 <pinref part="JP2" gate="G$1" pin="4"/>
-<pinref part="JP3" gate="G$1" pin="4"/>
 <wire x1="149.86" y1="81.28" x2="165.1" y2="81.28" width="0.1524" layer="91"/>
+<pinref part="JP1" gate="G$1" pin="5"/>
 </segment>
 </net>
@@
 <wire x1="86.36" y1="96.52" x2="93.98" y2="96.52" width="0.1524" layer="91"/>
 <label x="91.44" y="96.52" size="1.778" layer="95"/>
+<pinref part="D1" gate="G$1" pin="C"/>
+<wire x1="104.14" y1="93.98" x2="104.14" y2="91.44" width="0.1524" layer="91"/>
+<wire x1="104.14" y1="91.44" x2="93.98" y2="91.44" width="0.1524" layer="91"/>
+<wire x1="93.98" y1="91.44" x2="93.98" y2="96.52" width="0.1524" layer="91"/>
 </segment>
 <segment>
@@
 <segment>
 <pinref part="U1" gate="G$1" pin="CS_M"/>
-<wire x1="73.66" y1="63.5" x2="83.82" y2="63.5" width="0.1524" layer="91"/>
 <label x="76.2" y="63.5" size="1.778" layer="95"/>
+<pinref part="R2" gate="G$1" pin="2"/>
+<wire x1="73.66" y1="63.5" x2="93.98" y2="63.5" width="0.1524" layer="91"/>
+<wire x1="93.98" y1="63.5" x2="93.98" y2="66.04" width="0.1524" layer="91"/>
 </segment>
 <segment>
@@
 </segment>
 <segment>
-<pinref part="JP3" gate="G$1" pin="3"/>
 <wire x1="165.1" y1="78.74" x2="160.02" y2="78.74" width="0.1524" layer="91"/>
 <label x="160.02" y="78.74" size="1.778" layer="95"/>
+<pinref part="JP1" gate="G$1" pin="6"/>
 </segment>
 </net>
@@
 <segment>
 <pinref part="JP2" gate="G$1" pin="7"/>
-<pinref part="JP3" gate="G$1" pin="7"/>
 <wire x1="149.86" y1="88.9" x2="165.1" y2="88.9" width="0.1524" layer="91"/>
 <label x="152.4" y="88.9" size="1.778" layer="95"/>
-</segment>
-</net>
+<pinref part="JP1" gate="G$1" pin="2"/>
+</segment>
+</net>
