File: Hardware/LSM9DS1/20160708_DWC_LSM9DS1.brd (EAGLE design)
At the start: 41.5 x 26.8 mm, 52 parts, among them U1 LSM9DS1, U2 LSM9DS1, U3 LSM9DS1, U4 LSM9DS1

Commit message: updated cam
Parts:
- renumbered U$1 to T1, U$2 to T2, U$3 to T3, U$4 to T4
