File: Hardware/Skin_Sensor/LPS25H.sch (KiCad schematic (older format))
At the start: 49 parts, among them SW1 SW_PUSH, U1 ADP7102, U2 ATSAMD21E18A, U3 AVRISP, U4 LSM9DS1, U5 LP5521YQ, X1 ABS06

Commit message: Fixed pour issues
Parts:
- C19: value 100nF -> 10uF
- C22: value 100nF -> 10nF
- C24, C25: value 4.7UF -> 1uF
- C26, C27: value 4.7UF -> 0.47uF
- R1: value 10k -> 330
- R10, R11, R12, R13, R4, R5, R6, R7, R8, R9: value RES -> 10k
Changed lines of the file:
@@
 P 7750 1150
 F 0 "R5" H 7800 1075 20  0000 C CNN
-F 1 "RES" H 7675 1200 20  0000 C CNN
+F 1 "10k" H 7675 1200 20  0000 C CNN
 F 2 "Resistors_SMD:R_0402" H 7750 1150 60  0001 C CNN
 F 3 "" H 7750 1150 60  0001 C CNN
@@
 P 10200 1200
 F 0 "R7" H 10250 1125 20  0000 C CNN
-F 1 "RES" H 10125 1250 20  0000 C CNN
+F 1 "10k" H 10125 1250 20  0000 C CNN
 F 2 "Resistors_SMD:R_0402" H 10200 1200 60  0001 C CNN
 F 3 "" H 10200 1200 60  0001 C CNN
@@
 P 7600 1150
 F 0 "R4" H 7650 1075 20  0000 C CNN
-F 1 "RES" H 7525 1200 20  0000 C CNN
+F 1 "10k" H 7525 1200 20  0000 C CNN
 F 2 "Resistors_SMD:R_0402" H 7600 1150 60  0001 C CNN
 F 3 "" H 7600 1150 60  0001 C CNN
@@
 P 10150 1600
 F 0 "R6" H 10200 1525 20  0000 C CNN
-F 1 "RES" H 10075 1650 20  0000 C CNN
+F 1 "10k" H 10075 1650 20  0000 C CNN
 F 2 "Resistors_SMD:R_0402" H 10150 1600 60  0001 C CNN
 F 3 "" H 10150 1600 60  0001 C CNN
@@
 P 5650 4650
 F 0 "R1" H 5700 4575 20  0000 C CNN
-F 1 "10k" H 5575 4700 20  0000 C CNN
+F 1 "330" H 5575 4700 20  0000 C CNN
 F 2 "Resistors_SMD:R_0402" H 5650 4650 60  0001 C CNN
 F 3 "" H 5650 4650 60  0001 C CNN
@@
 P 5800 2750
 F 0 "C22" H 5850 2675 20  0000 C CNN
-F 1 "100nF" H 5725 2800 20  0000 C CNN
+F 1 "10nF" H 5725 2800 20  0000 C CNN
 F 2 "Capacitors_SMD:C_0402" H 5800 2750 60  0001 C CNN
 F 3 "" H 5800 2750 60  0001 C CNN
@@
 P 5350 2750
 F 0 "C19" H 5400 2675 20  0000 C CNN
-F 1 "100nF" H 5275 2800 20  0000 C CNN
+F 1 "10uF" H 5275 2800 20  0000 C CNN
 F 2 "Capacitors_SMD:C_0402" H 5350 2750 60  0001 C CNN
 F 3 "" H 5350 2750 60  0001 C CNN
@@
 P 7450 2250
 F 0 "R8" H 7500 2175 20  0000 C CNN
-F 1 "RES" H 7375 2300 20  0000 C CNN
+F 1 "10k" H 7375 2300 20  0000 C CNN
 F 2 "Resistors_SMD:R_0402" H 7450 2250 60  0001 C CNN
 F 3 "" H 7450 2250 60  0001 C CNN
@@
 P 7550 2250
 F 0 "R9" H 7600 2175 20  0000 C CNN
-F 1 "RES" H 7475 2300 20  0000 C CNN
+F 1 "10k" H 7475 2300 20  0000 C CNN
 F 2 "Resistors_SMD:R_0402" H 7550 2250 60  0001 C CNN
 F 3 "" H 7550 2250 60  0001 C CNN
@@
 P 7650 2250
 F 0 "R10" H 7700 2175 20  0000 C CNN
-F 1 "RES" H 7575 2300 20  0000 C CNN
+F 1 "10k" H 7575 2300 20  0000 C CNN
 F 2 "Resistors_SMD:R_0402" H 7650 2250 60  0001 C CNN
 F 3 "" H 7650 2250 60  0001 C CNN
@@
 P 7750 2250
 F 0 "R11" H 7800 2175 20  0000 C CNN
-F 1 "RES" H 7675 2300 20  0000 C CNN
+F 1 "10k" H 7675 2300 20  0000 C CNN
 F 2 "Resistors_SMD:R_0402" H 7750 2250 60  0001 C CNN
 F 3 "" H 7750 2250 60  0001 C CNN
@@
 P 8700 2650
 F 0 "C26" H 8750 2575 20  0000 C CNN
-F 1 "4.7UF" H 8625 2700 20  0000 C CNN
+F 1 "0.47uF" H 8625 2700 20  0000 C CNN
 F 2 "Capacitors_SMD:C_0402" H 8700 2650 60  0001 C CNN
 F 3 "" H 8700 2650 60  0001 C CNN
@@
 P 8850 2900
 F 0 "C27" H 8900 2825 20  0000 C CNN
-F 1 "4.7UF" H 8775 2950 20  0000 C CNN
+F 1 "0.47uF" H 8775 2950 20  0000 C CNN
 F 2 "Capacitors_SMD:C_0402" H 8850 2900 60  0001 C CNN
 F 3 "" H 8850 2900 60  0001 C CNN
@@
 P 10250 2550
 F 0 "R13" H 10300 2475 20  0000 C CNN
-F 1 "RES" H 10175 2600 20  0000 C CNN
+F 1 "10k" H 10175 2600 20  0000 C CNN
 F 2 "Resistors_SMD:R_0402" H 10250 2550 60  0001 C CNN
 F 3 "" H 10250 2550 60  0001 C CNN
@@
 P 10150 2550
 F 0 "R12" H 10200 2475 20  0000 C CNN
-F 1 "RES" H 10075 2600 20  0000 C CNN
+F 1 "10k" H 10075 2600 20  0000 C CNN
 F 2 "Resistors_SMD:R_0402" H 10150 2550 60  0001 C CNN
 F 3 "" H 10150 2550 60  0001 C CNN
@@
 P 8550 2600
 F 0 "C25" H 8600 2525 20  0000 C CNN
-F 1 "4.7UF" H 8475 2650 20  0000 C CNN
+F 1 "1uF" H 8475 2650 20  0000 C CNN
 F 2 "Capacitors_SMD:C_0402" H 8550 2600 60  0001 C CNN
 F 3 "" H 8550 2600 60  0001 C CNN
@@
 P 8400 2600
 F 0 "C24" H 8450 2525 20  0000 C CNN
-F 1 "4.7UF" H 8325 2650 20  0000 C CNN
+F 1 "1uF" H 8325 2650 20  0000 C CNN
 F 2 "Capacitors_SMD:C_0402" H 8400 2600 60  0001 C CNN
 F 3 "" H 8400 2600 60  0001 C CNN

Commit message: Added sensor and cleaned up the board
Parts:
- added C15: sj2, _Fab_Footprint:SJ-2-1-no, symbol solder_jumper_2_1_no_conn
- added C28, C3: 100nF, Capacitors_SMD:C_0603, symbol CAP
- added P1: CONN_01X05, _Fab_Footprint:2.54mmX05, symbol CONN_01X05
- added R14: 100k, Resistors_SMD:R_0402, symbol RES
- added U6: DPS310, _CSL:8-LGA, symbol DPS310
- C11, C12: footprint Fab_Footprint:SJ-2-1-no -> _Fab_Footprint:SJ-2-1-no
- C16, C17, C18: footprint Fab_Footprint:WM1387x06-REC -> _Fab_Footprint:WM1387x06-REC
- D2: footprint Fab_Footprint:4-PLCC -> _Fab_Footprint:4-PLCC
- L1, L2: footprint Fab_Footprint:LPS25H -> _Fab_Footprint:LPS25H
- SW1: footprint Fab_Footprint:SPST-NO-TL3700 -> _Fab_Footprint:SPST-NO-TL3700
- U2: footprint Fab_Footprint:QFN-32-1EP_5x5mm_Pitch0.5mm -> _Fab_Footprint:QFN-32-1EP_5x5mm_Pitch0.5mm
- U3: footprint Fab_Footprint:TagConnectx06 -> _Fab_Footprint:TagConnectx06
- U4: footprint Fab_Footprint:LSM9DS1 -> _Fab_Footprint:LSM9DS1
- X1: footprint Fab_Footprint:ABS06 -> _Fab_Footprint:ABS06
Connections:
- net labels added: GND_EX, INT_EX, SCL_EX, SDA_EX, VDD_EX
- wire segments 299 -> 326
Other:
- note added: "Sensors"
- note added: "Testing A New Sensor"
- note removed: "Sensor"
- moved on the sheet: C10, C13, C14, C19, C20, C21, C22, C23, C24, C25, C26, C27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
